File: IR/Init.kicad_pcb (KiCad board)
At the start: 2 copper layers, 43 parts, among them J1 CONN_C1, J4 CONN_C3, J5 Conn_01x06_Female, J7 CONN_C2, J9 CONN_C4, U1 NE555, U2 LM324

Commit message: PCB prototype
Parts:
- added H1: MountingHole_Pad, MountingHole:MountingHole_3.2mm_M3_DIN965_Pad, F.Cu at (155.0, 55.0)
- added H2: MountingHole_Pad, MountingHole:MountingHole_3.2mm_M3_DIN965_Pad, F.Cu at (215.0, 95.0)
- added H3: MountingHole_Pad, MountingHole:MountingHole_3.2mm_M3_DIN965_Pad, F.Cu at (215.0, 55.0)
- added H4: MountingHole_Pad, MountingHole:MountingHole_3.2mm_M3_DIN965_Pad, F.Cu at (155.0, 95.0)
- moved C7 135.8 mm to (160.2, 64.6)
- moved R11 135.6 mm to (163.8, 64.5)
- moved U2 135.5 mm to (170.8, 52.0)
- moved J1 135.5 mm to (161.1, 96.5)
- moved C16 135.5 mm to (160.2, 62.0)
- moved C3 135.4 mm to (165.5, 91.5)
- moved D2 135.3 mm to (167.2, 64.6)
- moved R23 135.2 mm to (163.8, 62.0)
- moved D6 135.0 mm to (167.2, 62.0)
- moved D3 134.9 mm to (181.8, 64.5)
- moved Rmes1 134.9 mm to (160.8, 88.8)
- moved D8 134.8 mm to (181.8, 62.0)
- moved Rlim1 134.8 mm to (169.8, 98.5)
- moved R4 134.8 mm to (163.8, 88.8)
- moved C18 134.7 mm to (188.8, 62.0)
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Routing:
- net GND: track 195.5 -> 279.6 mm
- net +5V: track 237.8 -> 176.5 mm
- net C2: track 49.9 -> 74.1 mm
- net C4: track 32.1 -> 46.4 mm
- net C1: track 50.2 -> 62.4 mm
- net C3: track 30.4 -> 42.1 mm
- net Net-(C5-Pad1): track 60.1 -> 52.1 mm
- net Net-(C12-Pad1): track 40.5 -> 47.2 mm
- net Net-(C5-Pad2): track 10.00 -> 8.85 mm
- net Net-(C6-Pad1): track 19.9 -> 18.8 mm
- net Net-(C13-Pad2): track 9.77 -> 8.86 mm
- net Net-(C3-Pad2): track 9.88 -> 9.04 mm
- net Net-(J7-Pad3): track 5.37 -> 4.53 mm
- net Net-(C12-Pad2): track 9.77 -> 8.94 mm
- net Net-(J4-Pad3): track 5.46 -> 4.64 mm
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- added copper zone on B.Cu, net GND
- added copper zone on F.Cu, net GND
Other:
- board outline added: 70 x 50 mm
- board text added: "Robotronik-Init-2019"
