File: Main_PCB/init/init.sch (KiCad schematic (older format))
At the start: 15 parts, among them J1 Conn_01x06_Male, J2 Conn_01x02_Male, J3 Conn_01x02_Female, J4 Conn_01x02_Female, J5 Conn_01x04_Female, U1 L293D

Commit message: v2
Parts:
- added D3: D, Diode_THT:D_5KPW_P12.70mm_Horizontal, symbol Device:D
Connections:
- net +5V: no longer U1.8 (VCC2)
- net +BATT: now also U1.8 (VCC2), D3.1 (K); no longer J2.1 (Pin_1)
- new net: D3.2 (A), J2.1 (Pin_1)
Changed lines of the file:
@@
-$EndComp
-$Comp
-L power:PWR_FLAG #FLG0101
-U 1 1 5943E881
-P 5800 2000
-F 0 "#FLG0101" H 5800 2075 50  0001 C CNN
-F 1 "PWR_FLAG" H 5800 2150 50  0000 C CNN
-F 2 "" H 5800 2000 50  0001 C CNN
-F 3 "" H 5800 2000 50  0001 C CNN
-	1    5800 2000
-	1    0    0    -1
 $EndComp
 $Comp
@@
 L power:+BATT #PWR0104
 U 1 1 5D7A15B3
-P 2550 3850
-F 0 "#PWR0104" H 2550 3700 50  0001 C CNN
-F 1 "+BATT" H 2565 4023 50  0000 C CNN
-F 2 "" H 2550 3850 50  0001 C CNN
-F 3 "" H 2550 3850 50  0001 C CNN
-	1    2550 3850
+P 2900 3850
+F 0 "#PWR0104" H 2900 3700 50  0001 C CNN
+F 1 "+BATT" H 2915 4023 50  0000 C CNN
+F 2 "" H 2900 3850 50  0001 C CNN
+F 3 "" H 2900 3850 50  0001 C CNN
+	1    2900 3850
 	1    0    0    -1
 $EndComp
@@
 $EndComp
 Wire Wire Line
-	2550 3850 2550 3900
-Wire Wire Line
-	2550 3900 2250 3900
+	2900 3850 2900 3900
+Wire Wire Line
+	2900 3900 2650 3900
 $Comp
 L power:GND #PWR0106
@@
 	5200 2100 5200 2150
 Wire Wire Line
-	5900 2100 5800 2100
-Wire Wire Line
 	5500 2100 5500 2200
 Wire Wire Line
 	5500 2000 5500 2100
 Connection ~ 5500 2100
-Wire Wire Line
-	5800 2000 5800 2100
-Connection ~ 5800 2100
-Wire Wire Line
-	5800 2100 5500 2100
 $Comp
 L power:GND #PWR0110
@@
 Wire Wire Line
 	7900 2550 7900 2400
-Connection ~ 7900 2400
-Wire Wire Line
-	7900 2400 8100 2400
 Wire Wire Line
 	7500 3950 7400 3950
@@
 Wire Wire Line
 	9700 1750 9600 1750
+$Comp
+L power:+BATT #PWR01
+U 1 1 5D8EC8C6
+P 8400 2350
+F 0 "#PWR01" H 8400 2200 50  0001 C CNN
+F 1 "+BATT" H 8415 2523 50  0000 C CNN
+F 2 "" H 8400 2350 50  0001 C CNN
+F 3 "" H 8400 2350 50  0001 C CNN
+	1    8400 2350
+	1    0    0    -1
+$EndComp
+Wire Wire Line
+	8400 2350 8400 2400
+Wire Wire Line
+	8400 2400 8100 2400
+$Comp
+L Device:D D3
+U 1 1 5D8F4F51
+P 2500 3900
+F 0 "D3" H 2500 3684 50  0000 C CNN
+F 1 "D" H 2500 3775 50  0000 C CNN
+F 2 "Diode_THT:D_5KPW_P12.70mm_Horizontal" H 2500 3900 50  0001 C CNN
+F 3 "~" H 2500 3900 50  0001 C CNN
+	1    2500 3900
+	-1   0    0    1
+$EndComp
+Wire Wire Line
+	2350 3900 2250 3900
+Wire Wire Line
+	5500 2100 5900 2100
 $EndSCHEMATC
